File: PCB/nix3PowerFinal.brd (EAGLE design)
At the start: 153.7 x 43.5 mm, 53 parts, among them IC2 IC_PCF8563, IC3 REG1117, IC4 REG1117, Q2 MPSA56, Q3 IRF620, Q4 16MHz, U1 ATMEGA328, X1 K375M

Commit message: Fix pcb
Parts:
- L1: value (none) -> 470uH
- Q3: value IRF620 -> IRF630
Changed lines of the file:
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@@
 <attribute name="VALUE" x="111.887" y="5.715" size="1.27" layer="27" ratio="10" rot="R90"/>
 </element>
-<element name="Q3" library="transistor-fet" package="TO220" value="IRF620" x="123.825" y="13.335" smashed="yes">
+<element name="Q3" library="transistor-fet" package="TO220" value="IRF630" x="123.825" y="13.335" smashed="yes">
 <attribute name="VALUE" x="119.888" y="13.97" size="1.778" layer="27" ratio="10"/>
 </element>
@@
 <attribute name="VALUE" x="133.731" y="28.194" size="1.27" layer="27" ratio="10" rot="R270"/>
 </element>
-<element name="L1" library="inductor-neosid" package="BS11" value="" x="112.395" y="26.035" smashed="yes">
+<element name="L1" library="inductor-neosid" package="BS11" value="470uH" x="112.395" y="26.035" smashed="yes">
 <attribute name="MF" value="" x="112.395" y="26.035" size="1.778" layer="27" display="off"/>
 <attribute name="MPN" value="" x="112.395" y="26.035" size="1.778" layer="27" display="off"/>
