File: PCB/nix3PowerFinal.sch (EAGLE design)
At the start: 53 parts, among them IC2 IC_PCF8563, IC3 REG1117, IC4 REG1117, Q2 MPSA56, Q3 IRF620, Q4 16MHz, U1 ATMEGA328, X1 K375M

Commit message: Fix pcb
Parts:
- L1: value (none) -> 470uH
- Q3: value IRF620 -> IRF630
Changed lines of the file:
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@@
 <part name="D5" library="diode" deviceset="DIODE-" device="D-5" value="BAV21"/>
 <part name="Q2" library="transistor-pnp" deviceset="MPSA56*" device=""/>
-<part name="Q3" library="transistor-fet" deviceset="IRF620" device=""/>
+<part name="Q3" library="transistor-fet" deviceset="IRF620" device="" value="IRF630"/>
 <part name="R8" library="resistor" deviceset="R-EU_" device="0204/5" value="1k"/>
 <part name="GND17" library="supply1" deviceset="GND" device=""/>
@@
 <part name="C9" library="resistor" deviceset="C-EU" device="050-025X075" value="100n"/>
 <part name="GND21" library="supply1" deviceset="GND" device=""/>
-<part name="L1" library="inductor-neosid" deviceset="BS" device="11"/>
+<part name="L1" library="inductor-neosid" deviceset="BS" device="11" value="470uH"/>
 <part name="SUPPLY10" library="supply2" deviceset="+12V" device=""/>
 <part name="SUPPLY11" library="supply2" deviceset="V+" device="" value="V+170"/>
